Commit message: candidates

File: ur_tof_description/urdf/a_ur_with_tof.urdf.xacro (robot description, xacro)
@@ -9,4 +9,14 @@
   <xacro:arg name="safety_limits" default="true"/>
   <xacro:arg name="prefix" default=""/>
+  <!-- Which YAML, how many sensors to place, sampling step -->
+  <xacro:arg name="candidates_yaml" default="$(find ur_simulation_gazebo)/candidates.yaml"/>
+  <xacro:arg name="pick_n" default="10"/>
+  <xacro:arg name="stride"  default="1"/>
+  <!-- Sensor defaults -->
+  <xacro:arg name="tof_rate" default="15"/>
+  <xacro:arg name="tof_max_range" default="3.0"/>
+  <!-- Load YAML (dict with keys: spacing_m, offset_m, candidate_count, candidates:[...]) -->
+  <xacro:property name="CANDS" value="${load_yaml(candidates_yaml)}"/>
+  <xacro:property name="LIST"  value="${CANDS['candidates']}"/>
   <!-- define dummy world link -->
   <link name="world"/>
@@ -27,8 +37,19 @@
   </xacro:ur_robot>
   <!-- Attach ToF sensors -->
-  <xacro:tof_sensor name="tof_wrist"   parent="wrist_3_link" xyz="0 0 0.10" rpy="0 0 0"  max_range="3.0" rate="15"/>
-  <xacro:tof_sensor name="tof_forearm" parent="forearm_link" xyz="0 0.05 0" rpy="0 1.57 0" max_range="3.0" rate="15"/>
-  <xacro:tof_sensor name="tof_shoulder" parent="shoulder_link" xyz="0.08 0 0" rpy="0 0 0" max_range="3.0" rate="15"/>
-  <xacro:tof_sensor name="tof_random" parent="forearm_link" xyz="0.5751823100486696 0.10664301745697961 0.11340798336935547" rpy="-1.574195687342217 -0.7603830563373393 0.7627287824310365" max_range="3.0" rate="15"/>
+  <!-- Auto-attach ToF sensors from YAML -->
+  <xacro:for each="it" in="${enumerate(LIST)}">
+    <xacro:property name="i" value="${it[0]}"/>
+    <xacro:property name="c" value="${it[1]}"/>
+    <!-- simple selection: every 'stride'-th candidate, up to pick_n -->
+    <xacro:if value="${i % int(stride) == 0 and i &lt; int(pick_n)}">
+      <xacro:tof_sensor
+        name="tof_${i}"
+        parent="${c['link']}"
+        xyz="${'{} {} {}'.format(c['xyz'][0], c['xyz'][1], c['xyz'][2])}"
+        rpy="${'{} {} {}'.format(c['rpy'][0], c['rpy'][1], c['rpy'][2])}"
+        max_range="$(arg tof_max_range)"
+        rate="$(arg tof_rate)"/>
+    </xacro:if>
+  </xacro:for>
   <!-- Gazebo ROS 2 Control -->
   <gazebo>
