Commit message: big voxels yay

File: ur_tof_description/urdf/ur_with_tof.urdf.xacro (robot description, xacro)
@@ -24,5 +24,5 @@
       safety_k_position="20"
       sim_gazebo="true">
-    <origin xyz="0 0 0" rpy="0 0 0"/>
+    <origin xyz="0 0 0.25" rpy="0 0 0"/>
   </xacro:ur_robot>
   <!-- Attach ToF sensors (auto-generated) -->
