Commit message: working sensor setup

File: ur_tof_description/urdf/sensors/tof_sensor.xacro (robot description, xacro)
@@ -1,5 +1,11 @@
 <?xml version="1.0"?>
 <robot xmlns:xacro="http://www.ros.org/wiki/xacro">
-  <xacro:macro name="tof_sensor" params="name parent xyz:='0 0 0' rpy:='0 0 0' min_range:=0.01 max_range:=2.0 rate:=30">
+  <!--
+    Simulates a VL53L7CX ToF array (~8x8 beams)
+    - Visible in Gazebo
+    - No collision geometry
+    - Publishes PointCloud2 on /<name>/points
+  -->
+  <xacro:macro name="tof_sensor" params="name parent xyz:='0 0 0' rpy:='0 0 0' min_range:=0.03 max_range:=3.5 rate:=15">
     <link name="${name}_link">
       <visual>
@@ -10,11 +16,8 @@
         </material>
       </visual>
-      <collision>
-        <geometry><cylinder radius="0.01" length="0.03"/></geometry>
-      </collision>
       <inertial>
         <origin xyz="0 0 0" rpy="0 0 0"/>
         <mass value="0.001"/>
-        <inertia ixx="1e-6" ixy="0.0" ixz="0.0" iyy="1e-6" iyz="0.0" izz="1e-6"/>
+        <inertia ixx="1e-6" ixy="0" ixz="0" iyy="1e-6" iyz="0" izz="1e-6"/>
       </inertial>
     </link>
@@ -26,14 +29,31 @@
     <gazebo reference="${name}_link">
       <sensor name="${name}_sensor" type="ray">
+        <always_on>true</always_on>
+        <visualize>true</visualize>
         <update_rate>${rate}</update_rate>
         <ray>
-          <scan><horizontal><samples>1</samples><resolution>1</resolution><min_angle>0.0</min_angle><max_angle>0.0</max_angle></horizontal></scan>
-          <range><min>${min_range}</min><max>${max_range}</max><resolution>0.001</resolution></range>
+          <scan>
+            <horizontal>
+              <samples>8</samples>
+              <resolution>1</resolution>
+              <min_angle>-0.523599</min_angle>  <!-- -30° -->
+              <max_angle> 0.523599</max_angle>  <!--  30° -->
+            </horizontal>
+            <vertical>
+              <samples>8</samples>
+              <resolution>1</resolution>
+              <min_angle>-0.523599</min_angle>
+              <max_angle> 0.523599</max_angle>
+            </vertical>
+          </scan>
+          <range>
+            <min>${min_range}</min>
+            <max>${max_range}</max>
+            <resolution>0.001</resolution>
+          </range>
         </ray>
         <plugin name="${name}_plugin" filename="libgazebo_ros_ray_sensor.so">
-          <ros>
-            <remapping>~/out:=/${name}/range</remapping>
-          </ros>
-          <output_type>sensor_msgs/Range</output_type>
+          <output_type>sensor_msgs/PointCloud2</output_type>
+          <frame_name>${name}_link</frame_name>
         </plugin>
       </sensor>

File: ur_tof_description/urdf/ur_with_tof.urdf.xacro (robot description, xacro)
@@ -3,13 +3,13 @@
   <!-- include UR base macros -->
   <xacro:include filename="$(find ur_description)/urdf/ur_macro.xacro"/>
-  <!-- include our sensor macro -->
+  <!-- include sensor macro -->
   <xacro:include filename="$(find ur_tof_description)/urdf/sensors/tof_sensor.xacro"/>
-  <!-- passthrough args that ur_simulation_gazebo already sets -->
+  <!-- passthrough args -->
   <xacro:arg name="ur_type" default="ur10"/>
   <xacro:arg name="safety_limits" default="true"/>
   <xacro:arg name="prefix" default=""/>
-  <!-- defining dummy world link -->
+  <!-- define dummy world link -->
   <link name="world"/>
-  <!-- Instantiate the UR robot (files depend on ur_type) -->
+  <!-- Instantiate the UR robot -->
   <xacro:ur_robot
       name="ur"
@@ -26,7 +26,13 @@
     <origin xyz="0 0 0" rpy="0 0 0"/>
   </xacro:ur_robot>
-  <!-- Attach ToF sensors to UR links; adjust positions as you like -->
-  <xacro:tof_sensor name="tof_wrist"   parent="wrist_3_link" xyz="0 0 0.10" rpy="0 0 0"  max_range="3.0" rate="30"/>
-  <xacro:tof_sensor name="tof_forearm" parent="forearm_link" xyz="0 0.05 0" rpy="0 1.57 0" max_range="2.0" rate="30"/>
-  <xacro:tof_sensor name="tof_shoulder" parent="shoulder_link" xyz="0.08 0 0" rpy="0 0 0" max_range="2.0" rate="20"/>
+  <!-- Attach ToF sensors -->
+  <xacro:tof_sensor name="tof_wrist"   parent="wrist_3_link" xyz="0 0 0.10" rpy="0 0 0"  max_range="3.0" rate="15"/>
+  <xacro:tof_sensor name="tof_forearm" parent="forearm_link" xyz="0 0.05 0" rpy="0 1.57 0" max_range="3.0" rate="15"/>
+  <xacro:tof_sensor name="tof_shoulder" parent="shoulder_link" xyz="0.08 0 0" rpy="0 0 0" max_range="3.0" rate="15"/>
+  <!-- Gazebo ROS 2 Control -->
+  <gazebo>
+    <plugin name="gazebo_ros2_control" filename="libgazebo_ros2_control.so">
+      <parameters>$(find ur_simulation_gazebo)/config/ur_controllers.yaml</parameters>
+    </plugin>
+  </gazebo>
 </robot>

Commit message: sensor xacro generator

File: ur_tof_description/urdf/sensors/tof_sensor.xacro (robot description, xacro)
@@ -10,5 +10,5 @@
     <link name="${name}_link">
       <visual>
-        <origin xyz="0 0 0.015" rpy="0 0 0"/>
+        <origin xyz="0.015 0 0" rpy="0 1.5708 0"/>
         <geometry><cylinder radius="0.01" length="0.03"/></geometry>
         <material name="${name}_mat">

File: ur_tof_description/urdf/ur_with_tof.urdf.xacro (robot description, xacro)
@@ -26,9 +26,15 @@
     <origin xyz="0 0 0" rpy="0 0 0"/>
   </xacro:ur_robot>
-  <!-- Attach ToF sensors -->
-  <xacro:tof_sensor name="tof_wrist"   parent="wrist_3_link" xyz="0 0 0.10" rpy="0 0 0"  max_range="3.0" rate="15"/>
-  <xacro:tof_sensor name="tof_forearm" parent="forearm_link" xyz="0 0.05 0" rpy="0 1.57 0" max_range="3.0" rate="15"/>
-  <xacro:tof_sensor name="tof_shoulder" parent="shoulder_link" xyz="0.08 0 0" rpy="0 0 0" max_range="3.0" rate="15"/>
-  <xacro:tof_sensor name="tof_random" parent="forearm_link" xyz="0.5751823100486696 0.10664301745697961 0.11340798336935547" rpy="-1.574195687342217 -0.7603830563373393 0.7627287824310365" max_range="3.0" rate="15"/>
+  <!-- Attach ToF sensors (auto-generated) -->
+  <xacro:tof_sensor name="tof_0" parent="base_link_inertia" xyz="-0.0797764151 0.00555363643 0.0336772195" rpy="-3.05105088 -0.000590753406 3.05105088" max_range="3" rate="15"/>
+  <xacro:tof_sensor name="tof_40" parent="base_link_inertia" xyz="0.00503601732 0.0610580514 -0.005" rpy="3.14159265 1.57079633 0" max_range="3" rate="15"/>
+  <xacro:tof_sensor name="tof_80" parent="forearm_link" xyz="-0.612050918 -0.0315296491 0.104844364" rpy="2.47463437 -1.09343012e-16 -2.47463437" max_range="3" rate="15"/>
+  <xacro:tof_sensor name="tof_120" parent="forearm_link" xyz="-0.53277249 -0.0410818426 0.0199500915" rpy="1.58535161 0.593151936 -1.58535161" max_range="3" rate="15"/>
+  <xacro:tof_sensor name="tof_160" parent="forearm_link" xyz="-0.427460762 -0.0107982347 0.094957204" rpy="1.57079749 -1.32533766 -1.57079749" max_range="3" rate="15"/>
+  <xacro:tof_sensor name="tof_200" parent="forearm_link" xyz="-0.31601453 0.045634711 0.0334473055" rpy="-1.57079628 0.343584055 1.57079628" max_range="3" rate="15"/>
+  <xacro:tof_sensor name="tof_240" parent="forearm_link" xyz="-0.194615769 -0.0468064701 0.0377606567" rpy="1.57079629 0.245472372 -1.57079629" max_range="3" rate="15"/>
+  <xacro:tof_sensor name="tof_280" parent="forearm_link" xyz="-0.0898612315 0.031500361 0.0120712985" rpy="-1.57079585 0.834520285 1.57079585" max_range="3" rate="15"/>
+  <xacro:tof_sensor name="tof_320" parent="forearm_link" xyz="-0.033049631 -0.00648535593 -0.00645266636" rpy="5.14279111e-05 1.1638215 -5.14279111e-05" max_range="3" rate="15"/>
+  <xacro:tof_sensor name="tof_360" parent="forearm_link" xyz="0.0275892508 0.055733588 0.100482886" rpy="-1.10378604 -0.000616611391 1.10378604" max_range="3" rate="15"/>
   <!-- Gazebo ROS 2 Control -->
   <gazebo>
